File: Hardware/Qwiic_IMU_Bonobo.brd (EAGLE design)
At the start: 30.5 x 25.4 mm, 37 parts, among them J2 SMD, J3 PTH, J4 SMD, J6 SPI, U2 BNO080, Y1 32.768kHz

Commit message: added bno080 to sfe lib
Parts:
- U2: device BNO080:LGA-28 -> SparkFun-IC-Special-Function:LGA-28
- moved LOGO2 41.9 mm to (0.00, -11.4)
- moved FRAME1 12.6 mm to (-11.4, -8.89)
Other:
- board text added: "A. England"
Changed lines of the file:
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@@
 <layer number="20" name="Dimension" color="15" fill="1" visible="yes" active="yes"/>
 <layer number="21" name="tPlace" color="16" fill="1" visible="yes" active="yes"/>
-<layer number="22" name="bPlace" color="14" fill="1" visible="no" active="yes"/>
+<layer number="22" name="bPlace" color="14" fill="1" visible="yes" active="yes"/>
 <layer number="23" name="tOrigins" color="15" fill="1" visible="yes" active="yes"/>
-<layer number="24" name="bOrigins" color="15" fill="1" visible="no" active="yes"/>
+<layer number="24" name="bOrigins" color="15" fill="1" visible="yes" active="yes"/>
 <layer number="25" name="tNames" color="7" fill="1" visible="yes" active="yes"/>
 <layer number="26" name="bNames" color="7" fill="1" visible="no" active="yes"/>
@@
 <layer number="49" name="Reference" color="7" fill="1" visible="no" active="yes"/>
 <layer number="50" name="dxf" color="7" fill="1" visible="no" active="yes"/>
-<layer number="51" name="tDocu" color="6" fill="1" visible="no" active="yes"/>
+<layer number="51" name="tDocu" color="6" fill="1" visible="yes" active="yes"/>
 <layer number="52" name="bDocu" color="7" fill="1" visible="no" active="yes"/>
 <layer number="53" name="tGND_GNDA" color="7" fill="9" visible="no" active="no"/>
@@
 <wire x1="7.62" y1="17.78" x2="22.86" y2="17.78" width="0.1524" layer="22"/>
 <wire x1="22.86" y1="17.78" x2="22.86" y2="20.32" width="0.1524" layer="22"/>
-<text x="10.16" y="-17.78" size="1.778" layer="51" font="vector" ratio="15">N. Seidle</text>
+<text x="19.05" y="-8.89" size="1.778" layer="51" font="vector">N. Seidle</text>
+<text x="19.05" y="-11.43" size="1.778" layer="51" font="vector">A. England</text>
 </plain>
 <attributes>
@@
 <element name="J2" library="SparkX" package="1X04_1MM_RA" value="SMD" x="5.08" y="12.7" rot="R270"/>
 <element name="J3" library="SparkX" package="1X04_NO_SILK" value="PTH" x="11.43" y="1.27"/>
-<element name="FRAME1" library="SparkFun-Aesthetics" package="CREATIVE_COMMONS" value="FRAME-LETTER" x="-20.32" y="-17.78"/>
+<element name="FRAME1" library="SparkFun-Aesthetics" package="CREATIVE_COMMONS" value="FRAME-LETTER" x="-11.43" y="-8.89"/>
 <element name="U$2" library="SparkFun-Aesthetics" package="SFE_LOGO_NAME_FLAME_.1" value="SFE_LOGO_NAME_FLAME.1_INCH" x="18.796" y="15.367"/>
 <element name="C4" library="SparkFun-Capacitors" package="0603" value="0.1uF" x="14.224" y="7.62" rot="R270">
@@
 <element name="LOGO1" library="SparkFun-Aesthetics" package="OSHW-LOGO-MINI" value="OSHW-LOGOMINI" x="27.94" y="2.54" rot="MR0"/>
 <element name="U$1" library="SparkFun-Aesthetics" package="SFE_LOGO_NAME_.1" value="SFE_LOGO_NAME.1_INCH" x="21.209" y="8.89" rot="MR0"/>
-<element name="U2" library="BNO080" package="LGA-28" value="BNO080" x="15.24" y="12.7" rot="R90"/>
+<element name="U2" library="SparkFun-IC-Special-Function" package="LGA-28" value="BNO080" x="15.24" y="12.7" rot="R90">
+<attribute name="PROD_ID" value="SEN-13947" x="15.24" y="12.7" size="1.778" layer="27" rot="R90" display="off"/>
+</element>
 <element name="C1" library="SparkFun-Capacitors" package="0603" value="0.1uF" x="12.319" y="7.62" rot="R270">
 <attribute name="PROD_ID" value="CAP-00810" x="12.319" y="7.62" size="1.778" layer="27" font="vector" ratio="15" rot="R270" display="off"/>
@@
 <attribute name="PROD_ID" value="CAP-07876" x="12.7" y="16.51" size="1.778" layer="27" font="vector" ratio="15" rot="R90" display="off"/>
 </element>
-<element name="LOGO2" library="SparkFun-Aesthetics" package="REVISION" value="REVISION" x="-40.64" y="-21.59"/>
+<element name="LOGO2" library="SparkFun-Aesthetics" package="REVISION" value="REVISION" x="0" y="-11.43"/>
 </elements>
 <signals>
