File: Hardware/Qwiic_IMU_Bonobo.brd (EAGLE design)
At the start: 30.5 x 25.4 mm, 85 parts, among them J2 SMD, J3 PTH, J4 SMD, J6 SPI, U2 BNO080, Y1 32.768kHz

Commit message: updated to Nates BNO080
Parts:
- added U$59: (no value), Qwiic#Label#Full#M#png (6):QWIIC#LABEL#FULL#M#PNG

Commit message: pre review
Parts:
- added LOGO2: REVISION, SparkFun-Aesthetics:REVISION
- moved FRAME1 12.7 mm to (-12.7, -7.62)
Other:
- board text added: "A. England"
- board text added: "v10"
- board text removed: "V10"
Changed lines of the file:
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@@
 <layer number="20" name="Dimension" color="15" fill="1" visible="yes" active="yes"/>
 <layer number="21" name="tPlace" color="16" fill="1" visible="yes" active="yes"/>
-<layer number="22" name="bPlace" color="14" fill="1" visible="yes" active="yes"/>
+<layer number="22" name="bPlace" color="14" fill="1" visible="no" active="yes"/>
 <layer number="23" name="tOrigins" color="15" fill="1" visible="yes" active="yes"/>
-<layer number="24" name="bOrigins" color="15" fill="1" visible="yes" active="yes"/>
-<layer number="25" name="tNames" color="7" fill="1" visible="no" active="yes"/>
+<layer number="24" name="bOrigins" color="15" fill="1" visible="no" active="yes"/>
+<layer number="25" name="tNames" color="7" fill="1" visible="yes" active="yes"/>
 <layer number="26" name="bNames" color="7" fill="1" visible="no" active="yes"/>
 <layer number="27" name="tValues" color="7" fill="1" visible="no" active="yes"/>
@@
 <layer number="43" name="vRestrict" color="2" fill="10" visible="no" active="yes"/>
 <layer number="44" name="Drills" color="7" fill="1" visible="no" active="yes"/>
-<layer number="45" name="Holes" color="7" fill="1" visible="yes" active="yes"/>
+<layer number="45" name="Holes" color="7" fill="1" visible="no" active="yes"/>
 <layer number="46" name="Milling" color="3" fill="1" visible="no" active="yes"/>
 <layer number="47" name="Measures" color="7" fill="1" visible="no" active="yes"/>
 <layer number="48" name="Document" color="7" fill="1" visible="no" active="yes"/>
-<layer number="49" name="Reference" color="7" fill="1" visible="yes" active="yes"/>
+<layer number="49" name="Reference" color="7" fill="1" visible="no" active="yes"/>
 <layer number="50" name="dxf" color="7" fill="1" visible="no" active="yes"/>
-<layer number="51" name="tDocu" color="6" fill="1" visible="yes" active="yes"/>
+<layer number="51" name="tDocu" color="6" fill="1" visible="no" active="yes"/>
 <layer number="52" name="bDocu" color="7" fill="1" visible="no" active="yes"/>
 <layer number="53" name="tGND_GNDA" color="7" fill="9" visible="no" active="no"/>
@@
 <wire x1="30.48" y1="25.4" x2="30.48" y2="0" width="0.2032" layer="20"/>
 <wire x1="30.48" y1="0" x2="0" y2="0" width="0.2032" layer="20"/>
-<text x="2.413" y="1.27" size="1.27" layer="16" font="vector" ratio="15" rot="MR0" align="center">V10</text>
+<text x="2.413" y="1.27" size="1.27" layer="16" font="vector" ratio="15" rot="MR0" align="center">v10</text>
 <dimension x1="2.54" y1="22.86" x2="27.94" y2="22.86" x3="15.24" y3="31.75" textsize="1.27" textratio="15" layer="47" unit="inch"/>
 <dimension x1="0" y1="25.4" x2="0" y2="0" x3="-8.89" y3="12.7" textsize="1.27" textratio="15" layer="47" unit="inch"/>
@@
 <wire x1="3.038975" y1="19.38741875" x2="3.308384375" y2="19.297615625" width="0.1778" layer="22"/>
 <wire x1="7.62" y1="17.78" x2="22.86" y2="17.78" width="0.1524" layer="22"/>
-<text x="10.16" y="-17.78" size="1.778" layer="51" font="vector" ratio="15">N. Seidle</text>
+<text x="17.78" y="-7.62" size="1.778" layer="51" font="vector">N. Seidle</text>
 <dimension x1="6.35" y1="1.27" x2="6.35" y2="24.13" x3="-3.81" y3="12.7" textsize="1.27" textratio="15" layer="47" dtype="vertical" unit="inch"/>
 <dimension x1="8.89" y1="19.05" x2="8.89" y2="24.13" x3="-1.27" y3="21.59" textsize="1.27" textratio="15" layer="47" dtype="vertical" unit="inch"/>
+<text x="17.78" y="-10.16" size="1.778" layer="51" font="vector">A. England</text>
 </plain>
 <attributes>
@@
 <element name="J2" library="SparkX" package="1X04_1MM_RA" value="SMD" x="5.08" y="12.7" rot="R270"/>
 <element name="J3" library="SparkX" package="1X04_NO_SILK" value="PTH" x="11.43" y="1.27"/>
-<element name="FRAME1" library="SparkFun-Aesthetics" package="CREATIVE_COMMONS" value="FRAME-LETTER" x="-20.32" y="-17.78"/>
+<element name="FRAME1" library="SparkFun-Aesthetics" package="CREATIVE_COMMONS" value="FRAME-LETTER" x="-12.7" y="-7.62"/>
 <element name="C4" library="SparkFun-Capacitors" package="0603" value="0.1uF" x="14.224" y="7.62" rot="R270">
 <attribute name="PROD_ID" value="CAP-00810" x="14.224" y="7.62" size="1.778" layer="27" font="vector" ratio="15" rot="R270" display="off"/>
@@
 <element name="U$1" library="Labels-0_04" package="(PWR)" value="" x="25.781" y="15.875" rot="R90"/>
 <element name="U$59" library="Qwiic#Label#Full#M#png (6)" package="QWIIC#LABEL#FULL#M#PNG" value="" x="27.305" y="13.208" rot="MR0"/>
+<element name="LOGO2" library="SparkFun-Aesthetics" package="REVISION" value="REVISION" x="-33.02" y="-13.97"/>
 </elements>
 <signals>

Commit message: post design review
Parts:
- added JP1, JP5: FIDUCIALUFIDUCIAL, SparkFun:MICRO-FIDUCIAL
- moved JP2 59.2 mm to (-29.6, 0.89), flipped to the bottom
- moved U$39 58.9 mm to (-29.5, 18.0), flipped to the top
- moved R2 58.2 mm to (-29.1, 18.3), flipped to the bottom
- moved U$23 57.7 mm to (-28.8, 3.17), flipped to the bottom
- moved JP4 55.9 mm to (-27.9, 22.9), flipped to the bottom
- moved LOGO1 55.9 mm to (-27.9, 2.54), flipped to the top
- moved D1 55.1 mm to (-27.6, 18.3), flipped to the bottom
- moved U$59 54.6 mm to (-27.3, 13.2), flipped to the top
- moved R12 53.3 mm to (-26.7, 7.62), flipped to the bottom
- moved R13 53.3 mm to (-26.7, 2.54), flipped to the bottom
- moved SJ1 53.3 mm to (-26.7, 5.08), flipped to the bottom
- moved U$30 52.6 mm to (-26.3, 6.35), flipped to the top
- moved U$1 51.6 mm to (-25.8, 15.9), flipped to the bottom
- moved J4 50.8 mm to (-25.4, 12.7), flipped to the bottom
- moved U$44 49.0 mm to (-24.5, 13.5), flipped to the top
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Connections:
- net ADR/MOSI renamed ADDR/MOSI

Commit message: Adding panel files
Parts:
- moved JP1 59.2 mm to (29.6, 0.89), flipped to the bottom
- moved JP2 59.2 mm to (29.6, 0.89), flipped to the top
- moved U$39 58.9 mm to (29.5, 18.0), flipped to the bottom
- moved R2 58.2 mm to (29.1, 18.3), flipped to the top
- moved U$23 57.7 mm to (28.8, 3.17), flipped to the top
- moved JP4 55.9 mm to (27.9, 22.9), flipped to the top
- moved LOGO1 55.9 mm to (27.9, 2.54), flipped to the bottom
- moved D1 55.1 mm to (27.6, 18.3), flipped to the top
- moved U$59 54.6 mm to (27.3, 13.2), flipped to the bottom
- moved R12 53.3 mm to (26.7, 7.62), flipped to the top
- moved R13 53.3 mm to (26.7, 2.54), flipped to the top
- moved SJ1 53.3 mm to (26.7, 5.08), flipped to the top
- moved U$30 52.6 mm to (26.3, 6.35), flipped to the bottom
- moved U$1 51.6 mm to (25.8, 15.9), flipped to the top
- moved J4 50.8 mm to (25.4, 12.7), flipped to the top
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