File: Hardware/Qwiic_IMU_Bonobo.sch (EAGLE design)
At the start: 37 parts, among them J2 SMD, J3 PTH, J4 SMD, J6 SPI, U2 BNO080, Y1 32.768kHz

Commit message: added bno080 to sfe lib
Parts:
- U2: device BNO080:BNO080 -> SparkFun-IC-Special-Function:BNO080
Changed lines of the file:
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@@
 <part name="LOGO1" library="SparkFun-Aesthetics" deviceset="OSHW-LOGO" device="MINI"/>
 <part name="U$1" library="SparkFun-Aesthetics" deviceset="SFE_LOGO_NAME" device=".1_INCH" value="SFE_LOGO_NAME.1_INCH"/>
-<part name="U2" library="BNO080" deviceset="BNO080" device=""/>
+<part name="U2" library="SparkFun-IC-Special-Function" deviceset="BNO080" device=""/>
 <part name="C1" library="SparkFun-Capacitors" deviceset="0.1UF" device="-0603-25V-(+80/-20%)" value="0.1uF"/>
 <part name="GND3" library="SparkFun" deviceset="GND" device=""/>

Commit message: adding Nates BNO080
Parts:
- removed LOGO2: REVISION, SparkFun-Aesthetics:REVISION
- removed U$1: SFE_LOGO_NAME.1_INCH, SparkFun-Aesthetics:SFE_LOGO_NAME.1_INCH
- removed U$2: SFE_LOGO_NAME_FLAME.1_INCH, SparkFun-Aesthetics:SFE_LOGO_NAME_FLAME.1_INCH
- added D1: RED, SparkFun-LED:LED-RED0603
- added LOGO4: SFE_LOGO_FLAME.1_INCH, SparkFun-Aesthetics:SFE_LOGO_FLAME.1_INCH
- added LOGO5: SFE_LOGO_NAME_FLAME.1_INCH, SparkFun-Aesthetics:SFE_LOGO_NAME_FLAME.1_INCH
- added R2: 1k, SparkFun-Resistors:1KOHM-0603-1/10W-1%
Connections:
- new net N$3: D1.C, R2.2
- net 3.3V: now also D1.A
- net GND: now also R2.1
Other:
- note added: "Power"
- note added: "X10"
- note removed: "A. England"
- note removed: "v01"
- moved on the sheet: R7, R8, SJ3, SJ4
Changed lines of the file:
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@@
 <part name="GND7" library="SparkFun" deviceset="GND" device=""/>
 <part name="FRAME1" library="SparkFun-Aesthetics" deviceset="FRAME-LETTER" device=""/>
-<part name="U$2" library="SparkFun-Aesthetics" deviceset="SFE_LOGO_NAME_FLAME" device=".1_INCH" value="SFE_LOGO_NAME_FLAME.1_INCH"/>
 <part name="C4" library="SparkFun-Capacitors" deviceset="0.1UF" device="-0603-25V-(+80/-20%)" value="0.1uF"/>
 <part name="SUPPLY8" library="SparkFun-PowerSymbols" deviceset="3.3V" device=""/>
@@
 <part name="GND8" library="SparkFun" deviceset="GND" device=""/>
 <part name="LOGO1" library="SparkFun-Aesthetics" deviceset="OSHW-LOGO" device="MINI"/>
-<part name="U$1" library="SparkFun-Aesthetics" deviceset="SFE_LOGO_NAME" device=".1_INCH" value="SFE_LOGO_NAME.1_INCH"/>
 <part name="U2" library="SparkFun-IC-Special-Function" deviceset="BNO080" device=""/>
 <part name="C1" library="SparkFun-Capacitors" deviceset="0.1UF" device="-0603-25V-(+80/-20%)" value="0.1uF"/>
@@
 <part name="C5" library="SparkFun-Capacitors" deviceset="22PF" device="-0603-50V-5%" value="22pF"/>
 <part name="GND14" library="SparkFun" deviceset="GND" device=""/>
-<part name="LOGO2" library="SparkFun-Aesthetics" deviceset="REVISION" device=""/>
+<part name="LOGO4" library="SparkFun-Aesthetics" deviceset="SFE_LOGO_FLAME" device=".1_INCH"/>
+<part name="LOGO5" library="SparkFun-Aesthetics" deviceset="SFE_LOGO_NAME_FLAME" device=".1_INCH"/>
+<part name="D1" library="SparkFun-LED" deviceset="LED-RED" device="0603" value="RED"/>
+<part name="SUPPLY3" library="SparkFun-PowerSymbols" deviceset="3.3V" device=""/>
+<part name="R2" library="SparkFun-Resistors" deviceset="1KOHM" device="-0603-1/10W-1%" value="1k"/>
+<part name="GND15" library="SparkFun" deviceset="GND" device=""/>
 </parts>
 <sheets>
@@
 <plain>
 <text x="170.434" y="11.43" size="2.54" layer="94">N. Seidle</text>
-<text x="237.744" y="7.366" size="2.54" layer="94">v01</text>
+<text x="237.744" y="7.366" size="2.54" layer="94">X10</text>
 <text x="7.62" y="132.08" size="1.778" layer="97">7-Bit I2C Address Jumper</text>
 <text x="10.16" y="127" size="1.778" layer="97">Closed = 0x4A</text>
@@
 <wire x1="147.32" y1="91.44" x2="147.32" y2="35.56" width="0.2032" layer="97"/>
 <wire x1="93.98" y1="91.44" x2="93.98" y2="0" width="0.2032" layer="97"/>
-<text x="174.752" y="6.858" size="2.54" layer="94">A. England</text>
+<text x="240.792" y="159.258" size="1.778" layer="97" rot="R90">Power</text>
 </plain>
 <instances>
@@
 <instance part="FRAME1" gate="G$1" x="0" y="0"/>
 <instance part="FRAME1" gate="V" x="147.32" y="0"/>
-<instance part="U$2" gate="G$1" x="2.54" y="0"/>
 <instance part="C4" gate="G$1" x="185.42" y="127"/>
 <instance part="SUPPLY8" gate="G$1" x="66.04" y="43.18" rot="MR0"/>
 <instance part="J4" gate="G$1" x="55.88" y="35.56"/>
 <instance part="GND8" gate="1" x="66.04" y="27.94" rot="MR0"/>
-<instance part="LOGO1" gate="G$1" x="76.2" y="12.7"/>
-<instance part="U$1" gate="G$1" x="1.27" y="0.508"/>
+<instance part="LOGO1" gate="G$1" x="121.92" y="22.86"/>
 <instance part="U2" gate="U1" x="124.46" y="132.08"/>
 <instance part="C1" gate="G$1" x="144.78" y="106.68"/>
@@
 <instance part="R6" gate="G$1" x="58.42" y="149.86" rot="MR90"/>
 <instance part="SUPPLY11" gate="G$1" x="58.42" y="157.48" rot="MR0"/>
-<instance part="R7" gate="G$1" x="213.36" y="149.86" rot="R90"/>
-<instance part="SUPPLY12" gate="G$1" x="213.36" y="172.72"/>
-<instance part="R8" gate="G$1" x="228.6" y="149.86" rot="R90"/>
-<instance part="SUPPLY13" gate="G$1" x="228.6" y="172.72"/>
-<instance part="GND11" gate="1" x="213.36" y="139.7"/>
-<instance part="GND12" gate="1" x="228.6" y="139.7"/>
-<instance part="SJ3" gate="1" x="213.36" y="165.1" rot="MR270"/>
-<instance part="SJ4" gate="1" x="228.6" y="165.1" rot="MR270"/>
+<instance part="R7" gate="G$1" x="205.74" y="149.86" rot="R90"/>
+<instance part="SUPPLY12" gate="G$1" x="205.74" y="172.72"/>
+<instance part="R8" gate="G$1" x="220.98" y="149.86" rot="R90"/>
+<instance part="SUPPLY13" gate="G$1" x="220.98" y="172.72"/>
+<instance part="GND11" gate="1" x="205.74" y="139.7"/>
+<instance part="GND12" gate="1" x="220.98" y="139.7"/>
+<instance part="SJ3" gate="1" x="205.74" y="165.1" rot="MR270"/>
+<instance part="SJ4" gate="1" x="220.98" y="165.1" rot="MR270"/>
 <instance part="R9" gate="G$1" x="157.48" y="147.32" rot="R90"/>
 <instance part="R10" gate="G$1" x="165.1" y="147.32" rot="R90"/>
@@
 <instance part="C5" gate="G$1" x="165.1" y="111.76"/>
 <instance part="GND14" gate="1" x="165.1" y="104.14"/>
-<instance part="LOGO2" gate="G$1" x="148.59" y="7.112"/>
+<instance part="LOGO4" gate="G$1" x="99.06" y="20.32"/>
+<instance part="LOGO5" gate="G$1" x="17.78" y="0"/>
+<instance part="D1" gate="G$1" x="233.68" y="165.1"/>
+<instance part="SUPPLY3" gate="G$1" x="233.68" y="172.72"/>
+<instance part="R2" gate="G$1" x="233.68" y="149.86" rot="R90"/>
+<instance part="GND15" gate="1" x="233.68" y="139.7"/>
 </instances>
 <busses>
@@
 <pinref part="SJ3" gate="1" pin="1"/>
 <pinref part="SUPPLY12" gate="G$1" pin="3.3V"/>
-<wire x1="213.36" y1="172.72" x2="213.36" y2="170.18" width="0.1524" layer="91"/>
+<wire x1="205.74" y1="172.72" x2="205.74" y2="170.18" width="0.1524" layer="91"/>
 </segment>
 <segment>
 <pinref part="SJ4" gate="1" pin="1"/>
 <pinref part="SUPPLY13" gate="G$1" pin="3.3V"/>
-<wire x1="228.6" y1="172.72" x2="228.6" y2="170.18" width="0.1524" layer="91"/>
+<wire x1="220.98" y1="172.72" x2="220.98" y2="170.18" width="0.1524" layer="91"/>
 </segment>
 <segment>
@@
 <wire x1="205.74" y1="50.8" x2="205.74" y2="68.58" width="0.1524" layer="91"/>
 <pinref part="SUPPLY2" gate="G$1" pin="3.3V"/>
+</segment>
+<segment>
+<pinref part="D1" gate="G$1" pin="A"/>
+<pinref part="SUPPLY3" gate="G$1" pin="3.3V"/>
+<wire x1="233.68" y1="172.72" x2="233.68" y2="167.64" width="0.1524" layer="91"/>
 </segment>
 </net>
@@
 <pinref part="GND11" gate="1" pin="GND"/>
 <pinref part="R7" gate="G$1" pin="1"/>
-<wire x1="213.36" y1="144.78" x2="213.36" y2="142.24" width="0.1524" layer="91"/>
+<wire x1="205.74" y1="144.78" x2="205.74" y2="142.24" width="0.1524" layer="91"/>
 </segment>
 <segment>
 <pinref part="GND12" gate="1" pin="GND"/>
 <pinref part="R8" gate="G$1" pin="1"/>
-<wire x1="228.6" y1="144.78" x2="228.6" y2="142.24" width="0.1524" layer="91"/>
+<wire x1="220.98" y1="144.78" x2="220.98" y2="142.24" width="0.1524" layer="91"/>
 </segment>
 <segment>
@@
 <wire x1="104.14" y1="144.78" x2="101.6" y2="144.78" width="0.1524" layer="91"/>
 <label x="101.6" y="144.78" size="1.27" layer="95" rot="R180" xref="yes"/>
+</segment>
+<segment>
+<pinref part="R2" gate="G$1" pin="1"/>
+<pinref part="GND15" gate="1" pin="GND"/>
+<wire x1="233.68" y1="142.24" x2="233.68" y2="144.78" width="0.1524" layer="91"/>
 </segment>
 </net>
@@
 </segment>
 <segment>
-<label x="210.82" y="157.48" size="1.27" layer="95" rot="R180" xref="yes"/>
-<wire x1="210.82" y1="157.48" x2="213.36" y2="157.48" width="0.1524" layer="91"/>
+<label x="203.2" y="157.48" size="1.27" layer="95" rot="R180" xref="yes"/>
+<wire x1="203.2" y1="157.48" x2="205.74" y2="157.48" width="0.1524" layer="91"/>
 <pinref part="R7" gate="G$1" pin="2"/>
-<wire x1="213.36" y1="157.48" x2="213.36" y2="154.94" width="0.1524" layer="91"/>
+<wire x1="205.74" y1="157.48" x2="205.74" y2="154.94" width="0.1524" layer="91"/>
 <pinref part="SJ3" gate="1" pin="2"/>
-<wire x1="213.36" y1="157.48" x2="213.36" y2="160.02" width="0.1524" layer="91"/>
-<junction x="213.36" y="157.48"/>
+<wire x1="205.74" y1="157.48" x2="205.74" y2="160.02" width="0.1524" layer="91"/>
+<junction x="205.74" y="157.48"/>
 </segment>
 <segment>
@@
 </segment>
 <segment>
-<label x="226.06" y="157.48" size="1.27" layer="95" rot="R180" xref="yes"/>
-<wire x1="226.06" y1="157.48" x2="228.6" y2="157.48" width="0.1524" layer="91"/>
+<label x="218.44" y="157.48" size="1.27" layer="95" rot="R180" xref="yes"/>
+<wire x1="218.44" y1="157.48" x2="220.98" y2="157.48" width="0.1524" layer="91"/>
 <pinref part="R8" gate="G$1" pin="2"/>
-<wire x1="228.6" y1="157.48" x2="228.6" y2="154.94" width="0.1524" layer="91"/>
+<wire x1="220.98" y1="157.48" x2="220.98" y2="154.94" width="0.1524" layer="91"/>
 <pinref part="SJ4" gate="1" pin="2"/>
-<wire x1="228.6" y1="160.02" x2="228.6" y2="157.48" width="0.1524" layer="91"/>
-<junction x="228.6" y="157.48"/>
+<wire x1="220.98" y1="160.02" x2="220.98" y2="157.48" width="0.1524" layer="91"/>
+<junction x="220.98" y="157.48"/>
 </segment>
 <segment>
@@
 </segment>
 </net>
+<net name="N$3" class="0">
+<segment>
+<pinref part="D1" gate="G$1" pin="C"/>
+<pinref part="R2" gate="G$1" pin="2"/>
+<wire x1="233.68" y1="154.94" x2="233.68" y2="160.02" width="0.1524" layer="91"/>
+</segment>
+</net>

Commit message: updated to Nates BNO080
Changed lines of the file:
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@@
 <instance part="C5" gate="G$1" x="165.1" y="111.76"/>
 <instance part="GND14" gate="1" x="165.1" y="104.14"/>
-<instance part="LOGO4" gate="G$1" x="99.06" y="20.32"/>
+<instance part="LOGO4" gate="G$1" x="50.292" y="12.446"/>
 <instance part="LOGO5" gate="G$1" x="17.78" y="0"/>
 <instance part="D1" gate="G$1" x="233.68" y="165.1"/>

Commit message: pre review
Parts:
- added LOGO2: REVISION, SparkFun-Aesthetics:REVISION
Other:
- note added: "A. England"
- note added: "v10"
- note removed: "X10"
Changed lines of the file:
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@@
 <part name="R2" library="SparkFun-Resistors" deviceset="1KOHM" device="-0603-1/10W-1%" value="1k"/>
 <part name="GND15" library="SparkFun" deviceset="GND" device=""/>
+<part name="LOGO2" library="SparkFun-Aesthetics" deviceset="REVISION" device=""/>
 </parts>
 <sheets>
@@
 <plain>
 <text x="170.434" y="11.43" size="2.54" layer="94">N. Seidle</text>
-<text x="237.744" y="7.366" size="2.54" layer="94">X10</text>
+<text x="237.744" y="7.366" size="2.54" layer="94">v10</text>
 <text x="7.62" y="132.08" size="1.778" layer="97">7-Bit I2C Address Jumper</text>
 <text x="10.16" y="127" size="1.778" layer="97">Closed = 0x4A</text>
@@
 <wire x1="93.98" y1="91.44" x2="93.98" y2="0" width="0.2032" layer="97"/>
 <text x="240.792" y="159.258" size="1.778" layer="97" rot="R90">Power</text>
+<text x="174.498" y="7.366" size="2.54" layer="94">A. England</text>
 </plain>
 <instances>
@@
 <instance part="R2" gate="G$1" x="233.68" y="149.86" rot="R90"/>
 <instance part="GND15" gate="1" x="233.68" y="139.7"/>
+<instance part="LOGO2" gate="G$1" x="148.59" y="7.366"/>
 </instances>
 <busses>

Commit message: post design review
Parts:
- added JP1, JP5: FIDUCIALUFIDUCIAL, SparkFun:FIDUCIALUFIDUCIAL
Connections:
- net ADR/MOSI renamed ADDR/MOSI
Other:
- note added: "Supply Voltage: 2.4V-3.6V"
- moved on the sheet: R3, SJ2
Changed lines of the file:
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@@
 <part name="GND15" library="SparkFun" deviceset="GND" device=""/>
 <part name="LOGO2" library="SparkFun-Aesthetics" deviceset="REVISION" device=""/>
+<part name="JP1" library="SparkFun" deviceset="FIDUCIAL" device="UFIDUCIAL"/>
+<part name="JP5" library="SparkFun" deviceset="FIDUCIAL" device="UFIDUCIAL"/>
 </parts>
 <sheets>
@@
 <text x="170.434" y="11.43" size="2.54" layer="94">N. Seidle</text>
 <text x="237.744" y="7.366" size="2.54" layer="94">v10</text>
-<text x="7.62" y="132.08" size="1.778" layer="97">7-Bit I2C Address Jumper</text>
-<text x="10.16" y="127" size="1.778" layer="97">Closed = 0x4A</text>
-<text x="10.16" y="129.54" size="1.778" layer="97">Open (default) = 0x4B</text>
+<text x="5.08" y="132.08" size="1.778" layer="97">7-Bit I2C Address Jumper</text>
+<text x="7.62" y="127" size="1.778" layer="97">Closed = 0x4A</text>
+<text x="7.62" y="129.54" size="1.778" layer="97">Open (default) = 0x4B</text>
 <text x="198.628" y="112.268" size="2.54" layer="97">PS0
  0
@@
 <text x="39.878" y="85.852" size="2.54" layer="97" align="center">2</text>
 <wire x1="0" y1="91.44" x2="93.98" y2="91.44" width="0.2032" layer="97"/>
-<wire x1="93.98" y1="91.44" x2="147.32" y2="91.44" width="0.2032" layer="97"/>
-<wire x1="147.32" y1="91.44" x2="248.92" y2="91.44" width="0.2032" layer="97"/>
-<wire x1="147.32" y1="91.44" x2="147.32" y2="35.56" width="0.2032" layer="97"/>
-<wire x1="93.98" y1="91.44" x2="93.98" y2="0" width="0.2032" layer="97"/>
+<wire x1="93.98" y1="91.44" x2="147.32" y2="91.44" width="0.2032" layer="97" style="longdash"/>
+<wire x1="147.32" y1="91.44" x2="248.92" y2="91.44" width="0.2032" layer="97" style="longdash"/>
+<wire x1="147.32" y1="91.44" x2="147.32" y2="35.56" width="0.2032" layer="97" style="longdash"/>
+<wire x1="93.98" y1="91.44" x2="93.98" y2="0" width="0.2032" layer="97" style="longdash"/>
 <text x="240.792" y="159.258" size="1.778" layer="97" rot="R90">Power</text>
 <text x="174.498" y="7.366" size="2.54" layer="94">A. England</text>
+<text x="109.22" y="160.02" size="1.27" layer="97" font="vector">Supply Voltage: 2.4V-3.6V</text>
 </plain>
 <instances>
@@
 <instance part="SUPPLY9" gate="G$1" x="101.6" y="152.4"/>
 <instance part="GND9" gate="1" x="157.48" y="104.14"/>
-<instance part="GND10" gate="1" x="45.72" y="124.46" rot="MR0"/>
-<instance part="SJ2" gate="1" x="45.72" y="134.62" rot="MR90"/>
-<instance part="SUPPLY10" gate="G$1" x="45.72" y="157.48" rot="MR0"/>
-<instance part="R3" gate="G$1" x="45.72" y="149.86" rot="MR90"/>
+<instance part="GND10" gate="1" x="43.18" y="124.46" rot="MR0"/>
+<instance part="SJ2" gate="1" x="43.18" y="134.62" rot="MR90"/>
+<instance part="SUPPLY10" gate="G$1" x="43.18" y="157.48" rot="MR0"/>
+<instance part="R3" gate="G$1" x="43.18" y="149.86" rot="MR90"/>
 <instance part="R6" gate="G$1" x="58.42" y="149.86" rot="MR90"/>
 <instance part="SUPPLY11" gate="G$1" x="58.42" y="157.48" rot="MR0"/>
@@
 <instance part="GND15" gate="1" x="233.68" y="139.7"/>
 <instance part="LOGO2" gate="G$1" x="148.59" y="7.366"/>
+<instance part="JP1" gate="G$1" x="233.68" y="30.48"/>
+<instance part="JP5" gate="G$1" x="238.76" y="30.48"/>
 </instances>
 <busses>
@@
 </segment>
 <segment>
-<wire x1="45.72" y1="157.48" x2="45.72" y2="154.94" width="0.1524" layer="91"/>
+<wire x1="43.18" y1="157.48" x2="43.18" y2="154.94" width="0.1524" layer="91"/>
 <pinref part="SUPPLY10" gate="G$1" pin="3.3V"/>
 <pinref part="R3" gate="G$1" pin="2"/>
@@
 <wire x1="104.14" y1="114.3" x2="101.6" y2="114.3" width="0.1524" layer="91"/>
 <junction x="101.6" y="114.3"/>
-</segment>
-<segment>
-<wire x1="45.72" y1="127" x2="45.72" y2="129.54" width="0.1524" layer="91"/>
+<pinref part="U2" gate="U1" pin="CLKSEL0"/>
+<wire x1="104.14" y1="144.78" x2="101.6" y2="144.78" width="0.1524" layer="91"/>
+<wire x1="101.6" y1="144.78" x2="101.6" y2="116.84" width="0.1524" layer="91"/>
+<junction x="101.6" y="116.84"/>
+</segment>
+<segment>
+<wire x1="43.18" y1="127" x2="43.18" y2="129.54" width="0.1524" layer="91"/>
 <pinref part="GND10" gate="1" pin="GND"/>
 <pinref part="SJ2" gate="1" pin="1"/>
@@
 </segment>
 <segment>
-<pinref part="U2" gate="U1" pin="CLKSEL0"/>
-<wire x1="104.14" y1="144.78" x2="101.6" y2="144.78" width="0.1524" layer="91"/>
-<label x="101.6" y="144.78" size="1.27" layer="95" rot="R180" xref="yes"/>
-</segment>
-<segment>
 <pinref part="R2" gate="G$1" pin="1"/>
 <pinref part="GND15" gate="1" pin="GND"/>
@@
 </segment>
 </net>
-<net name="ADR/MOSI" class="0">
-<segment>
-<wire x1="104.14" y1="142.24" x2="45.72" y2="142.24" width="0.1524" layer="91"/>
-<wire x1="45.72" y1="139.7" x2="45.72" y2="142.24" width="0.1524" layer="91"/>
-<wire x1="45.72" y1="142.24" x2="45.72" y2="144.78" width="0.1524" layer="91"/>
-<junction x="45.72" y="142.24"/>
+<net name="ADDR/MOSI" class="0">
+<segment>
+<wire x1="104.14" y1="142.24" x2="50.8" y2="142.24" width="0.1524" layer="91"/>
+<wire x1="50.8" y1="142.24" x2="43.18" y2="142.24" width="0.1524" layer="91"/>
+<wire x1="43.18" y1="139.7" x2="43.18" y2="142.24" width="0.1524" layer="91"/>
+<wire x1="43.18" y1="142.24" x2="43.18" y2="144.78" width="0.1524" layer="91"/>
+<junction x="43.18" y="142.24"/>
 <pinref part="SJ2" gate="1" pin="2"/>
 <pinref part="R3" gate="G$1" pin="1"/>
 <pinref part="U2" gate="U1" pin="H_SA0/MOSI"/>
-<wire x1="45.72" y1="142.24" x2="43.18" y2="142.24" width="0.1524" layer="91"/>
-<label x="43.18" y="142.24" size="1.27" layer="95" rot="R180" xref="yes"/>
+<label x="50.8" y="144.78" size="1.27" layer="95" font="vector" rot="R90" xref="yes"/>
+<wire x1="50.8" y1="144.78" x2="50.8" y2="142.24" width="0.1524" layer="91"/>
+<junction x="50.8" y="142.24"/>
 </segment>
 <segment>
@@
 <segment>
 <pinref part="U2" gate="U1" pin="PS0/WAKE"/>
-<wire x1="104.14" y1="124.46" x2="101.6" y2="124.46" width="0.1524" layer="91"/>
-<label x="101.6" y="124.46" size="1.27" layer="95" rot="R180" xref="yes"/>
+<wire x1="104.14" y1="124.46" x2="99.06" y2="124.46" width="0.1524" layer="91"/>
+<label x="99.06" y="124.46" size="1.27" layer="95" rot="R180" xref="yes"/>
 </segment>
 <segment>
@@
 <segment>
 <pinref part="U2" gate="U1" pin="PS1"/>
-<wire x1="104.14" y1="121.92" x2="101.6" y2="121.92" width="0.1524" layer="91"/>
-<label x="101.6" y="121.92" size="1.27" layer="95" rot="R180" xref="yes"/>
+<wire x1="104.14" y1="121.92" x2="99.06" y2="121.92" width="0.1524" layer="91"/>
+<label x="99.06" y="121.92" size="1.27" layer="95" rot="R180" xref="yes"/>
 </segment>
 <segment>
@@
 <segment>
 <pinref part="U2" gate="U1" pin="!H_CS"/>
-<wire x1="104.14" y1="132.08" x2="101.6" y2="132.08" width="0.1524" layer="91"/>
-<label x="101.6" y="132.08" size="1.27" layer="95" rot="R180" xref="yes"/>
+<wire x1="104.14" y1="132.08" x2="99.06" y2="132.08" width="0.1524" layer="91"/>
+<label x="99.06" y="132.08" size="1.27" layer="95" rot="R180" xref="yes"/>
 </segment>
 <segment>
@@
 <segment>
 <pinref part="U2" gate="U1" pin="!H_INT"/>
-<wire x1="104.14" y1="134.62" x2="101.6" y2="134.62" width="0.1524" layer="91"/>
-<label x="101.6" y="134.62" size="1.27" layer="95" rot="R180" xref="yes"/>
-</segment>
-<segment>
+<wire x1="104.14" y1="134.62" x2="99.06" y2="134.62" width="0.1524" layer="91"/>
+<label x="99.06" y="134.62" size="1.27" layer="95" rot="R180" xref="yes"/>
+</segment>
+<segment>
